File: sensor_logger.kicad_pcb (KiCad board)
At the start: 4 copper layers, 41 x 41.1 mm, 60 parts, among them IC1 TPS560430X3FDBVR, IC2 ASM330LHHTR, J1 USB4125-GF-A-0190, J2 Conn_01x10, J3 UART, J4 ST-Link/V2, U1 STM32F411CEU6

Commit message: Updated PCB to be a 2-layer board with through-hole vias
Parts:
- R10, R13, R14, R15, R16, R2, R8, R9: moved to F.Cu
- moved LED5V 27.0 mm to (47.6, 49.2), turned to 0 degrees
- moved LED3V3 25.9 mm to (47.7, 52.7), turned to 0 degrees
- moved R14 22.0 mm to (51.5, 49.2), turned to 180 degrees
- moved R13 20.6 mm to (51.7, 52.8), turned to 180 degrees
- moved C10 10.1 mm to (78.9, 69.7)
- moved FWST 7.04 mm to (68.2, 36.4), turned to 90 degrees
- moved R15 5.47 mm to (71.8, 36.4)
- moved R16 4.25 mm to (79.3, 36.4)
- moved R8 3.87 mm to (74.9, 49.2), turned to 180 degrees
- moved G*** 3.44 mm to (66.3, 50.0), turned to 145 degrees
- moved R9 3.07 mm to (71.8, 50.0)
- moved ERROR 2.67 mm to (76.0, 36.4), turned to 90 degrees
- moved R10 2.19 mm to (68.5, 49.5)
- moved R2 1.98 mm to (66.2, 56.5), turned to -90 degrees
- moved C2 1.77 mm to (78.7, 66.1)
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- renumbered LED_3V3 to LED3V3, LED_5V to LED5V
Routing:
- net +3V3: track 69.4 -> 212.9 mm, vias 23 -> 6
- net USB_VBUS: track 46.4 -> 35.1 mm, vias 1 -> 0
- net /LEDs/FWST: track 14.7 -> 22.5 mm, vias 1 -> 4
- net /LEDs/ERROR: track 15.2 -> 22.2 mm, vias 1 -> 4
- net /STM logic/GPIO_EXTI1: track 25.9 -> 32.3 mm, vias 4 -> 2
- net /Headers/NRST: track 26.3 -> 32.3 mm
- net Net-(IC2-CS): track 6.89 -> 4.07 mm, vias 1 -> 0
- net /STM logic/SPI1_MISO: track 11.7 -> 9.16 mm, vias 2 -> 0
- net I2C1_SDA: track 29.8 -> 32.2 mm, vias 2 -> 4
- net /STM logic/GPIO_EXTI2: track 24.9 -> 27.0 mm, vias 2 -> 4
- net /STM logic/TFT_SDCS: track 13.8 -> 11.8 mm
- net Net-(LED_5V1-A): track 3.76 -> 2.17 mm, vias 1 -> 0
- net /STM logic/TFT_CS: track 12.5 -> 10.9 mm
- net /Headers/SYS_JTMS-SWDIO: track 11.5 -> 13.0 mm
- net /STM logic/TFT_BL: track 12.0 -> 10.5 mm
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- added copper zone on B.Cu, net GND
- removed copper zone on In2.Cu, net +3V3
- removed copper zone on In1.Cu, net GND
Other:
- copper layers 4 -> 2
